File: Pogo - Top V1/Pad - Bottom V1.kicad_pcb (KiCad board)
At the start: 2 copper layers, 101.5 x 101.5 mm, 1 part, among them J1 Conn_01x02_Socket

Commit message: Precautionary commit
Connections:
- J1 pad 1: unconnected-(J1-Pin_1-Pad1) -> GND
- J1 pad 2: unconnected-(J1-Pin_2-Pad2) -> +9V
Routing:
- net unconnected-(J1-Pin_1-Pad1): track 22.2 -> 0.00 mm, vias 4 -> 0
- net GND: track 0.00 -> 22.2 mm, vias 0 -> 4
- net unconnected-(J1-Pin_2-Pad2): track 18.9 -> 0.00 mm
- net +9V: track 0.00 -> 18.9 mm
- added copper zone on F.Cu, net +9V
- added copper zone on B.Cu, net GND
- removed copper zone on B.Cu, net unconnected-(J1-Pin_1-Pad1)
- removed copper zone on F.Cu, net unconnected-(J1-Pin_2-Pad2)
Changed lines of the file:
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@@
 	)
 	(net 0 "")
-	(net 1 "unconnected-(J1-Pin_1-Pad1)")
-	(net 2 "unconnected-(J1-Pin_2-Pad2)")
+	(net 1 "GND")
+	(net 2 "+9V")
 	(footprint "Connector_AMASS:AMASS_XT30U-M_1x02_P5.0mm_Vertical"
 		(layer "B.Cu")
@@
 			)
 		)
-		(property "Datasheet" ""
+		(property "Datasheet" "https://www.tme.com/Document/7d9d972ae3468777f69ec2ee99897652/XT30U-M.pdf"
 			(at 0 0 0)
 			(unlocked yes)
@@
 			)
 		)
-		(property "Description" "Generic connector, single row, 01x02, script generated"
+		(property "Description" "2 PIN XT30 Male"
 			(at 0 0 0)
 			(unlocked yes)
@@
 			)
 		)
+		(property "Mfr." "TME"
+			(at 0 0 180)
+			(unlocked yes)
+			(layer "B.Fab")
+			(hide yes)
+			(effects
+				(font
+					(size 1 1)
+					(thickness 0.15)
+				)
+				(justify mirror)
+			)
+		)
+		(property "Part #" "XT30U-M"
+			(at 0 0 180)
+			(unlocked yes)
+			(layer "B.Fab")
+			(hide yes)
+			(effects
+				(font
+					(size 1 1)
+					(thickness 0.15)
+				)
+				(justify mirror)
+			)
+		)
+		(property "Order Link" "https://www.tme.com/us/en-us/details/xt30u-m/dc-power-connectors/amass/"
+			(at 0 0 180)
+			(unlocked yes)
+			(layer "B.Fab")
+			(hide yes)
+			(effects
+				(font
+					(size 1 1)
+					(thickness 0.15)
+				)
+				(justify mirror)
+			)
+		)
+		(property "Price" "$0.626"
+			(at 0 0 180)
+			(unlocked yes)
+			(layer "B.Fab")
+			(hide yes)
+			(effects
+				(font
+					(size 1 1)
+					(thickness 0.15)
+				)
+				(justify mirror)
+			)
+		)
 		(property ki_fp_filters "Connector*:*_1x??_*")
 		(sheetname "Root")
-		(sheetfile "Pogo - Bottom V1.kicad_sch")
+		(sheetfile "Pogo - Top V1.kicad_sch")
 		(attr through_hole)
 		(fp_line
@@
 			(layers "*.Cu" "*.Mask")
 			(remove_unused_layers no)
-			(net 1 "unconnected-(J1-Pin_1-Pad1)")
+			(net 1 "GND")
 			(pinfunction "Pin_1")
 			(pintype "passive")
@@
 			(layers "*.Cu" "*.Mask")
 			(remove_unused_layers no)
-			(net 2 "unconnected-(J1-Pin_2-Pad2)")
+			(net 2 "+9V")
 			(pinfunction "Pin_2")
 			(pintype "passive")
@@
 	(zone
 		(net 2)
-		(net_name "unconnected-(J1-Pin_2-Pad2)")
+		(net_name "+9V")
 		(layer "F.Cu")
 		(hatch edge 0.5)
@@
 	(zone
 		(net 1)
-		(net_name "unconnected-(J1-Pin_1-Pad1)")
+		(net_name "GND")
 		(layer "B.Cu")
 		(hatch edge 0.5)
