File: Float Power Board V1/Float Power Board V1.kicad_sch (KiCad schematic)
At the start: 10 parts, among them J1 Conn_01x02_Socket

Commit message: V1 of Float Boards ... most likely :)
Parts:
- BT1, BT2, BT3, BT4, BT5, BT7: MANUFACTURER Keystone Electronics -> (none); MAXIMUM_PACKAGE_HEIGHT 5.38mm -> (none); Mfr. (none) -> Keystone Electronics; Order Link (none) -> https://www.digikey.com/en/products/detail/keystone-electro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; PARTREV 10.16.07 -> (none); Part # (none) -> 967; Price (none) -> $1.174; SNAPEDA_PN 967 -> (none); STANDARD Manufacturer Recommendations -> (none)
- BT6: MANUFACTURER Keystone Electronics -> (none); MAXIMUM_PACKAGE_HEIGHT 5.38mm -> (none); Mfr. (none) -> Keystone Electronics; Order Link (none) -> https://www.digikey.com/en/products/detail/keystone-electro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; PARTREV 10.16.07 -> (none); Price  (none) -> $1.174; SNAPEDA_PN 967 -> (none); STANDARD Manufacturer Recommendations -> (none)
- BT8: MANUFACTURER Keystone Electronics -> (none); MAXIMUM_PACKAGE_HEIGHT 5.38mm -> (none); Mfr. (none) -> Keystone Electronics; Order Link (none) -> https://www.digikey.com/en/products/detail/keystone-electro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; PARTREV 10.16.07 -> (none); Part # (none) -> 967; Price  (none) -> $1.174; SNAPEDA_PN 967 -> (none); STANDARD Manufacturer Recommendations -> (none)
- F1: Mfr. (none) -> Keystone Electronics; Order Link (none) -> https://www.digikey.com/en/products/detail/keystone-electro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; Part # (none) -> 3588; Price (none) -> $1.25
