File: Glass Squid V2/Glass Squid V2.kicad_sch (KiCad schematic)
At the start: 25 parts, among them J1 Conn_01x16, J2 Conn_01x12, J3 SM04B-GHS-TB, J4 Qwiic_Vertical, J5 B2B-XH-A-GU, J6 B2B-XH-A-GU, J7 Conn_01x02, J9 Conn_01x03, Q1 AOSS32136C, U1 DRV8871DDA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

Commit message: V1 of Float Boards ... most likely :)
Parts:
- J4: Mfr. (none) -> JST Sales America Inc.; Order Link (none) -> https://www.digikey.com/en/products/detail/jst-sales-americ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; PROD_ID CONN-14483 -> (none); Part # (none) -> BM04B-SRSS-TB; Price (none) -> $0.462; Vendor (none) -> Digikey
- J7: Mfr. (none) -> TE Connectivity AMP Connectors; Order Link (none) -> https://www.digikey.com/en/products/detail/te-connectivity-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; Part # (none) -> 215297-2; Price (none) -> $0.91; Vendor (none) -> DigiKey
- Q1: Mfr. (none) -> Alpha & Omega Semiconductor Inc.; Order Link (none) -> https://www.digikey.com/en/products/detail/alpha-omega-semi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; Part # (none) -> AOSS32136C; Price (none) -> $0.29; Vendor (none) -> DigiKey
Changed lines of the file:
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@@
 			)
 		)
-		(property "Datasheet" "~"
+		(property "Datasheet" "https://www.te.com/usa-en/product-215297-2.datasheet.pdf"
 			(at 124.46 125.73 0)
 			(effects
@@
 			)
 		)
-		(property "Description" "Generic connector, single row, 01x02, script generated (kicad-library-utils/schlib/autogen/connector/)"
+		(property "Description" "CONN RCPT 2POS 0.1 GOLD PCB"
+			(at 124.46 125.73 0)
+			(effects
+				(font
+					(size 1.27 1.27)
+				)
+				(hide yes)
+			)
+		)
+		(property "Mfr." "TE Connectivity AMP Connectors"
+			(at 124.46 125.73 0)
+			(effects
+				(font
+					(size 1.27 1.27)
+				)
+				(hide yes)
+			)
+		)
+		(property "Part #" "215297-2"
+			(at 124.46 125.73 0)
+			(effects
+				(font
+					(size 1.27 1.27)
+				)
+				(hide yes)
+			)
+		)
+		(property "Vendor" "DigiKey"
+			(at 124.46 125.73 0)
+			(effects
+				(font
+					(size 1.27 1.27)
+				)
+				(hide yes)
+			)
+		)
+		(property "Order Link" "https://www.digikey.com/en/products/detail/te-connectivity-amp-connectors/215297-2/2055922"
+			(at 124.46 125.73 0)
+			(effects
+				(font
+					(size 1.27 1.27)
+				)
+				(hide yes)
+			)
+		)
+		(property "Price" "$0.91"
 			(at 124.46 125.73 0)
 			(effects
@@
 			)
 		)
-		(property "PROD_ID" "CONN-14483"
-			(at 236.22 106.68 0)
+		(property "Mfr." "JST Sales America Inc."
+			(at 236.22 96.52 0)
+			(effects
+				(font
+					(size 1.27 1.27)
+				)
+				(hide yes)
+			)
+		)
+		(property "Part #" "BM04B-SRSS-TB"
+			(at 236.22 96.52 0)
+			(effects
+				(font
+					(size 1.27 1.27)
+				)
+				(hide yes)
+			)
+		)
+		(property "Vendor" "Digikey"
+			(at 236.22 96.52 0)
+			(effects
+				(font
+					(size 1.27 1.27)
+				)
+				(hide yes)
+			)
+		)
+		(property "Order Link" "https://www.digikey.com/en/products/detail/jst-sales-america-inc/BM04B-SRSS-TB/926696"
+			(at 236.22 96.52 0)
+			(effects
+				(font
+					(size 1.27 1.27)
+				)
+				(hide yes)
+			)
+		)
+		(property "Price" "$0.462"
+			(at 236.22 96.52 0)
 			(effects
 				(font
@@
 			)
 		)
-		(property "Datasheet" "AOSS32136C"
+		(property "Datasheet" "https://www.aosmd.com/res/datasheets/AOSS32136C.pdf"
 			(at 134.62 135.89 0)
 			(effects
@@
 			)
 		)
-		(property "Description" ""
+		(property "Description" "MOSFET N-CH 20V 6.5A SOT23-3"
 			(at 134.62 135.89 0)
 			(effects
+				(font
+					(size 1.27 1.27)
+				)
+				(hide yes)
+			)
+		)
+		(property "Mfr." "Alpha & Omega Semiconductor Inc."
+			(at 134.62 135.89 0)
+			(effects
+				(font
+					(size 1.27 1.27)
+				)
+				(hide yes)
+			)
+		)
+		(property "Part #" "AOSS32136C"
+			(at 134.62 135.89 0)
+			(effects
+				(font
+					(size 1.27 1.27)
+				)
+				(hide yes)
+			)
+		)
+		(property "Vendor" "DigiKey"
+			(at 134.62 135.89 0)
+			(effects
+				(font
+					(size 1.27 1.27)
+				)
+				(hide yes)
+			)
+		)
+		(property "Order Link" "https://www.digikey.com/en/products/detail/alpha-omega-semiconductor-inc/AOSS32136C/11567433"
+			(at 134.62 135.89 0)
+			(effects
+				(font
+					(size 1.27 1.27)
+				)
+				(hide yes)
+			)
+		)
+		(property "Price" "$0.29"
+			(at 134.62 135.89 0)
+			(effects
